File: eBook Feather Wing/E-Book Wing Rev C.brd (EAGLE design)
At the start: 77.5 x 112.3 mm, 100 parts, among them IC1 MCP23008/SO, IC2 23K256-I/SN, J1 MJ-3523-SMT, Q1 IRLML0100, SW1 SPDT_SWITCH

Commit message: restore calvino quote, final version of wing A1-03 submitted to OSH Park
Parts:
- moved U$45 4.14 mm to (66.1, 27.3)
Other:
- board text added: "``Da anni frequento questa biblioteca e la esploro volume per volume, scaffale per scaffale, ma potrei dimostrarvi che non ho fatto altro che portare avanti la lettura d'un unico libro.'' - Italo Calvino, `Se una notte d'inverno un viaggiatore'"
Changed lines of the file:
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@@
 <?xml version="1.0" encoding="utf-8"?>
 <!DOCTYPE eagle SYSTEM "eagle.dtd">
-<eagle version="9.5.1">
+<eagle version="9.4.2">
 <drawing>
 <settings>
@@
 <setting verticaltext="up"/>
 </settings>
-<grid distance="0.01" unitdist="inch" unit="inch" style="lines" multiple="1" display="no" altdistance="1" altunitdist="mil" altunit="mil"/>
+<grid distance="0.01" unitdist="inch" unit="inch" style="lines" multiple="1" display="no" altdistance="0.001" altunitdist="inch" altunit="mil"/>
 <layers>
 <layer number="1" name="Top" color="4" fill="1" visible="yes" active="yes"/>
@@
 <wire x1="-0.254" y1="2.286" x2="2.032" y2="0" width="0" layer="20" curve="90"/>
 <wire x1="74.93" y1="0" x2="77.216" y2="2.286" width="0" layer="20" curve="90"/>
+<text x="38.608" y="64.514" size="1.016" layer="21" font="vector" align="center">``Da anni frequento questa biblioteca
+e la esploro volume per volume, scaffale
+per scaffale, ma potrei dimostrarvi che
+non ho fatto altro che portare avanti
+la lettura d'un unico libro.''
+- Italo Calvino, `Se una notte d'inverno un viaggiatore'
+</text>
 </plain>
 <attributes>
@@
 <element name="U$48" library="My Stuff" package="OSO_ONELINE_125MIL" value="OSO_TEXTOSO_TEXT_ONELINE_125MIL" x="45.339" y="14.732" smashed="yes"/>
 <element name="U$44" library="My Stuff" package="OSO_GRAPHIC" value="OSO_GRAPHIC" x="3.81" y="13.081" smashed="yes"/>
-<element name="U$45" library="My Stuff" package="OSO_BEAR_750MIL" value="OSO_BEAR" x="61.976" y="27.178" smashed="yes"/>
+<element name="U$45" library="My Stuff" package="OSO_BEAR_750MIL" value="OSO_BEAR" x="66.1162" y="27.305" smashed="yes"/>
 <element name="FCS" library="E-Book Wing Rev C (WIP)" package="SOLDERJUMPER_OPEN" value="SOLDERJUMPER_OPEN" x="33.274" y="44.45" smashed="yes" rot="MR180">
 <attribute name="NAME" x="35.56" y="44.45" size="0.508" layer="26" font="vector" ratio="18" rot="MR90" align="center"/>
