File: eBook Feather Wing/OSO-BOWI-A1-05 (WIP).brd (EAGLE design)
At the start: 77.5 x 112.3 mm, 100 parts, among them IC1 MCP23008/SO, IC2 23K256-I/SN, J1 SJ-43514-SMT, Q1 IRLML0100, SW1 SPDT_SWITCH

Commit message: silkscreen updates to e-book wing
Parts:
- removed U$8: (no value), My Stuff:OSO_BEAR_525X750MIL_1000DPI
- added U$13: (no value), My Stuff:OSO_WORDMARK_125X1300MIL_1000DPI
- added U$15: (no value), My Stuff:OSO_BEAR_250X360MIL_1000DPI
- MS1: value MICROBUILDER_FEATHERWING_SMTDUAL -> MICROBUILDER_FEATHERWING_SMTDUAL_NOLINES; device My Stuff:MICROBUILDER_FEATHERWING_SMT2 -> My Stuff:MICROBUILDER_FEATHERWING_SMT2_NOLINES
- moved R2 6.12 mm to (11.9, 65.5)
- moved C1 5.01 mm to (11.9, 61.5)
- moved D1 4.44 mm to (11.9, 48.5)
- moved R1 4.19 mm to (11.9, 43.2)
- moved FID4 2.96 mm to (1.52, 105.2)
- moved GOLD_ORB_SM1 1.27 mm to (67.1, 4.83)
- moved D2 1.27 mm to (11.9, 70.9)
- moved R3 0.76 mm to (58.7, 44.5)
- moved R4 0.76 mm to (58.7, 41.9)
- moved L1 0.25 mm to (38.4, 77.2)
Routing:
- net A1_: track 10.0 -> 5.55 mm
- net A1: track 42.0 -> 46.3 mm
- net A2_: track 10.4 -> 6.76 mm
- net +3V3: track 369.8 -> 367.3 mm
- net EN: track 25.4 -> 26.7 mm
- net BTN_PREV: track 185.6 -> 184.6 mm
- net A2: track 65.4 -> 66.3 mm
- net SDA: track 79.2 -> 79.9 mm
- net SCL: track 77.9 -> 78.7 mm
- net SD_CS: track 58.3 -> 58.9 mm
Other:
- board text added: "BUILDING THE E-BOOK WING"
- board text added: "CC-BY-SA 4.0 (except the bear!)"
- board text added: "EXTRA PORTS (STEMMA/JST-PH)"
- board text added: "For 4.2'' screen, E-Paper driver is IL0398. ECS is chip select for display. EDC indicates if transmission is data or a command. EBSY: signal from display; low = busy (for IL0398). ERST: signal to display, pull low to reset driver."
- board text added: "NOTE: This project requires some surface mount soldering, but there's only one truly fine-pitched part (the flex connector for the e-paper display). A fine- tipped soldering iron, flux and wick should be sufficient for this build; all chips are wide-pitch SOIC, and all resistors and capacitors are 0805 or larger so you can place them by eye with fine tweezers. Still, all surface mount parts are o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"
- board text added: "The E-Book Wing by Joey Castillo @josecastillo. OSO logo & lazer bear by Joseph Devens, @DoctorDevens. Shout out to Adafruit, OSHPark, the GNU Unifont project and everyone who's helped along the way!! Designed with . in BK & TX."
- board text added: "The MCP23008 provides eight additional GPIO pins via the I2C interface. It connects to all buttons except for RESET. R3 and R4 are the pull-up resistors for, respectively, SDA and SCL. This chip is required to use the buttons. You can also configure it to emit an interrupt signal on the INT pin when one or more buttons change state."
- board text added: "The center port provides an I²C interface. The other two ports provide access to pins A1 and A2 via current limiting resistors R1 and R2. D1 & D2 are 3.6V zener diodes to protect pins from overvoltage: they shunt excess power to ground when the voltage exceeds their breakdown point."
- board text added: "These are the Feather's UART pins, plus a 3V pin to power something like a GPS. Use the TX/GND/RX trio to talk to another e-book; just rotate one end 180° so one device's TX signal is the other's RX signal."
- board text removed: "@josecastillo"
- board text removed: "CC-BY-SA 4.0"
- board text removed: "EXTRA PORTS (JST-PH)"
- board text removed: "The MCP23008 provides eight additional GPIO pins via the I2C interface. It connects to all buttons except for RESET. R3 and R4 are the pull-up resistors for, respectively, SDA and SCL. This chip is required to use the buttons, unless you just want a few wired directly to GPIO pads. Capacitor C3 filters power."
- board text removed: "The center port provides an I2C interface. The other two ports provide access to pins A1 and A2. D1 & D2 + R1 & R2 provide protection and current limiting."
- board text removed: "The e-paper panel has an on-board booster that generates the high(er) voltages needed to drive the display. The circuit on the left deals with the boost voltages. C10-C16 are filtering caps for the power pins (in and out)."
- board text removed: "These are the Feather's UART pins, plus a 3V pin if you need to power something like a GPS. Toss some right angle header on here, it might prove useful."
- board text removed: "``Da anni frequento questa biblioteca e la esploro volume per volume, scaffale per scaffale, ma potrei dimostrarvi che non ho fatto altro che portare avanti la lettura d'un unico libro.'' - Italo Calvino, `Se una notte d'inverno un viaggiatore'"
- board text removed: "by joey castillo"
