File: eBook Feather Wing/OSO-BOWI-A1-06.brd (EAGLE design)
At the start: 77.5 x 112.3 mm, 105 parts, among them IC1 MCP23008/SO, IC2 23K256-I/SN, J1 SJ-43514-SMT, Q1 IRLML0100, SW1 SPDT_SWITCH

Commit message: rotate OSO logo to match open book
Parts:
- moved U$44 0.63 mm to (3.81, 12.4), turned to 45 degrees
Changed lines of the file:
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@@
 <layer number="27" name="tValues" color="7" fill="1" visible="no" active="yes"/>
 <layer number="28" name="bValues" color="7" fill="1" visible="no" active="yes"/>
-<layer number="29" name="tStop" color="7" fill="3" visible="no" active="yes"/>
+<layer number="29" name="tStop" color="7" fill="3" visible="yes" active="yes"/>
 <layer number="30" name="bStop" color="7" fill="6" visible="no" active="yes"/>
 <layer number="31" name="tCream" color="7" fill="4" visible="no" active="yes"/>
@@
 <attribute name="NAME" x="58.674" y="6.223" size="0.8128" layer="52" font="vector" ratio="18" rot="MR0" align="center"/>
 </element>
-<element name="U$44" library="My Stuff" package="OSO_GRAPHIC" value="OSO_GRAPHIC" x="3.81" y="13.081" smashed="yes"/>
+<element name="U$44" library="My Stuff" package="OSO_GRAPHIC" value="OSO_GRAPHIC" x="3.81" y="12.446" smashed="yes" rot="R45"/>
 <element name="BCS" library="E-Book Wing Rev C (WIP)" package="SOLDERJUMPER_OPEN" value="SOLDERJUMPER_OPEN" x="33.274" y="44.45" smashed="yes" rot="MR180">
 <attribute name="NAME" x="35.56" y="44.45" size="0.6096" layer="26" font="vector" ratio="18" rot="MR90" align="center"/>
@@
 <wire x1="2.2956" y1="91.3226" x2="0.381" y2="89.408" width="0.1524" layer="16"/>
 <via x="0.381" y="89.408" extent="1-16" drill="0.254"/>
-<wire x1="0.381" y1="89.408" x2="0.381" y2="11.049" width="0.1524" layer="1"/>
-<wire x1="3.556" y1="7.874" x2="0.381" y2="11.049" width="0.1524" layer="1"/>
+<wire x1="0.381" y1="89.408" x2="0.2032" y2="89.2302" width="0.1524" layer="1"/>
+<wire x1="0.2032" y1="89.2302" x2="0.2032" y2="11.2268" width="0.1524" layer="1"/>
+<wire x1="3.556" y1="7.874" x2="0.2032" y2="11.2268" width="0.1524" layer="1"/>
 <wire x1="12.4968" y1="0.4572" x2="61.4172" y2="0.4572" width="0.1524" layer="16"/>
 <wire x1="71.5789125" y1="24.9568" x2="71.3434" y2="25.1923125" width="0.1524" layer="16"/>
