File: Tiny Book/OSO-TIBO-A1-03 (WIP).brd (EAGLE design)
At the start: 54.9 x 88.1 mm, 106 parts, among them J2 10118193-0001LF, Q1 DMG341, Q2 IRLML0100, SW2 SPDT_SWITCH, U1 AP2112-3.3, U2 MCP73831T-2ACI/OT, U3 ATSAMD51G18A-MUT, U4 GD25Q32C, U5 MAX4468EKAT, X1 JSTPH, X2 2x5 0.05" SWD

Commit message: bump revision
Routing:
- net +3V3: vias 23 -> 21
Changed lines of the file:
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@@
 <wire x1="10.16" y1="37.88" x2="8.924" y2="39.116" width="0.3048" layer="16"/>
 <contactref element="D8_NEOPIXEL" pad="2"/>
-<wire x1="3.429" y1="72.39" x2="17.272" y2="72.39" width="0.3048" layer="1"/>
 <via x="24.638" y="72.39" extent="1-16" drill="0.3048"/>
-<wire x1="20.066" y1="72.39" x2="24.638" y2="72.39" width="0.3048" layer="1"/>
 <wire x1="24.638" y1="72.39" x2="32.35215" y2="72.39" width="0.3048" layer="16"/>
 <wire x1="6.916" y1="86.499" x2="6.916" y2="85.54" width="0.3048" layer="16"/>
@@
 <wire x1="13.65" y1="39.116" x2="12.446" y2="37.912" width="0.3048" layer="16"/>
 <via x="12.446" y="37.338" extent="1-16" drill="0.3048"/>
-<via x="20.066" y="72.39" extent="1-16" drill="0.3048"/>
-<wire x1="20.066" y1="72.39" x2="17.272" y2="72.39" width="0.3048" layer="16"/>
-<via x="17.272" y="72.39" extent="1-16" drill="0.3048"/>
 <via x="21.5392" y="59.944" extent="1-16" drill="0.3048"/>
 <wire x1="21.402" y1="55.372" x2="19.878" y2="53.848" width="0.3048" layer="16"/>
@@
 <wire x1="46.95918125" y1="76.454" x2="45.30018125" y2="78.113" width="0.3048" layer="16"/>
 <wire x1="50.58025" y1="76.454" x2="46.95918125" y2="76.454" width="0.3048" layer="16"/>
+<wire x1="3.429" y1="72.39" x2="24.638" y2="72.39" width="0.3048" layer="1"/>
 </signal>
 <signal name="GDR">
