File: eBook Feather Wing/OSO-BOWI-A1-06-KICAD/OSO-BOWI-A1-06.kicad_pcb (KiCad board)
At the start: 2 copper layers, 77.5 x 112.3 mm, 105 parts, among them IC1 MCP23008_SO, IC2 23K256-I/SN, IC3 MICROBUILDER_SPIFLASH_SOIC8, J1 SJ-43514-SMT, Q1 IRLML0100, SW1 SPDT_SWITCH

Commit message: Revised E-Book Wing silkscreen labels.
Addressing comment for the solder jumpers on the E-Book Wing that had silkscreen labels, such as TX1/RX1/ECS1 etc, where the number 1 was appended after the original name, which was crowding the labels and making the text less readable. The affected files are updated.
Other:
- board text added: "AREF"
- board text added: "BAT"
- board text added: "BCS"
- board text added: "EBSY"
- board text added: "ECS"
- board text added: "EDC"
- board text added: "EN"
- board text added: "ERST"
- board text added: "INT"
- board text added: "MISO"
- board text added: "MOSI"
- board text added: "RST"
- board text added: "SCK"
- board text added: "SDCS"
- board text added: "SRCS"
- board text added: "USB"
